File: hw/AA_P_CtrlBd.kicad_pcb (KiCad board)
At the start: 2 copper layers, 92 parts, among them J1 1x2 Pin Hdr, J10 AES-Option_A-B, J11 1x3 Pin Hdr, J12 1x3 Pin Hdr, J13 AES-Option_A-B, J14 1x3 Pin Hdr, J15 20-RBN, J16 1x3 Pin Hdr, J17 20-RBN, J18 1x3 Pin Hdr, J19 1x3 Pin Hdr, J2 SERVO-BAT (10-12V), J20 1x3 Pin Hdr, J21 1x3 Pin Hdr, J22 1x3 Pin Hdr, J23 1x3 Pin Hdr, J24 Conn_01x04, J25 Conn_01x04, J3 USB-C-Conn, J4 1x2 Pin Hdr, J5 1x2 Pin Hdr, J6 1x2 Pin Hdr, J7 1x3 Pin Hdr, J8 Conn_02x04_Odd_Even, J9 1x2 Pin Hdr, Q1 DMG2305UX, U1 TLV70033_SOT23-5, U10 74LS138, U11 74AHCT1G125, U2 BTS51202, U3 FT231XS, U4 AES-MCP23S08-E/SO, U5 74LVC1G10, U6 74AHCT1G125, U7 AES-Pico, U8 74LS138

Commit message: CTRL-BD-Pico: v1.0 to send for PCB.
Parts:
- removed C7: 4.7n, Capacitor_SMD:C_0603_1608Metric_Pad1.08x0.95mm_HandSolder
- removed R17, R18, R19, R20, R21, R22, R23, R24: 18k, Resistor_SMD:R_0805_2012Metric_Pad1.20x1.40mm_HandSolder
- added C16: 0.1u, Capacitor_SMD:C_0603_1608Metric_Pad1.08x0.95mm_HandSolder, F.Cu at (170.8, 42.2)
- added C19: 0.1u, Capacitor_SMD:C_0603_1608Metric_Pad1.08x0.95mm_HandSolder, F.Cu at (169.4, 47.9)
- added C21: 0.1u, Capacitor_SMD:C_0603_1608Metric_Pad1.08x0.95mm_HandSolder, F.Cu at (189.2, 47.4)
- added C22: T47u, Capacitor_Tantalum_SMD:CP_EIA-3528-21_Kemet-B_Pad1.50x2.35mm_HandSolder, F.Cu at (179.6, 45.2)
- added G1: LOGO, AES_Library:SILKY-DESIGN-logo-0_50-AES, F.Cu at (170.2, 138.4)
- added G1: LOGO, AES_Library:SILKY-DESIGN-logo-0_50-AES, B.Cu at (153.5, 117.6)
- added H1: M3, MountingHole:MountingHole_3.2mm_M3_ISO7380, F.Cu at (93.2, 142.5)
- added H2: M3, MountingHole:MountingHole_3.2mm_M3_ISO7380, F.Cu at (194.8, 142.5)
- added H3: M3, MountingHole:MountingHole_3.2mm_M3_ISO7380, F.Cu at (194.8, 40.9)
- added H4: M3, MountingHole:MountingHole_3.2mm_M3_ISO7380, F.Cu at (93.2, 40.9)
- added J26: HDR 1x4 Pin, Connector_PinHeader_2.54mm:PinHeader_1x04_P2.54mm_Vertical, F.Cu at (193.3, 136.9)
- added J27: JST-B4B-ZR 4P 1.5, Connector_Wuerth:Wuerth_WR-WTB_64800411622_1x04_P1.50mm_Vertical, F.Cu at (193.3, 131.6)
- added J28: HR-DF13-4P 1.25, Connector_Hirose:Hirose_DF13-04P-1.25DSA_1x04_P1.25mm_Vertical, F.Cu at (193.3, 124.5)
- added J29: HDR 2x10 Odd/Even, Connector_PinHeader_2.54mm:PinHeader_2x10_P2.54mm_Vertical, B.Cu at (138.4, 136.1)
- added J30: HDR 1x3 Pin, Connector_PinHeader_2.54mm:PinHeader_1x03_P2.54mm_Vertical, F.Cu at (195.2, 81.3)
- added J31: HDR 1x3 Pin, Connector_PinHeader_2.54mm:PinHeader_1x03_P2.54mm_Vertical, F.Cu at (195.2, 76.7)
- added J32: HDR 1x3 Pin, Connector_PinHeader_2.54mm:PinHeader_1x03_P2.54mm_Vertical, F.Cu at (195.2, 72.1)
- added J33: HDR 1x3 Pin, Connector_PinHeader_2.54mm:PinHeader_1x03_P2.54mm_Vertical, F.Cu at (195.2, 67.6)
- added J34: HDR 2x10 Odd/Even, Connector_PinHeader_2.54mm:PinHeader_2x10_P2.54mm_Vertical, F.Cu at (192.7, 109.3)
- added J35: HR DF13-2P, Connector_Hirose:Hirose_DF13-02P-1.25DSA_1x02_P1.25mm_Vertical, F.Cu at (186.1, 62.5)
- added J36: HR DF13-2P, Connector_Hirose:Hirose_DF13-02P-1.25DSA_1x02_P1.25mm_Vertical, F.Cu at (186.1, 55.9)
- added J37: HDR 1x10, Connector_PinHeader_2.54mm:PinHeader_1x10_P2.54mm_Vertical, F.Cu at (195.2, 109.3)
- added J38: Molex KK-254 AE-6410_1x03, Connector_Molex:Molex_KK-254_AE-6410-03A_1x03_P2.54mm_Vertical, F.Cu at (189.0, 116.6)
- added JP4: HDR 1x2 Pin, Connector_PinHeader_2.54mm:PinHeader_1x02_P2.54mm_Vertical, F.Cu at (171.6, 61.3)
- added JP5: HDR 1x2 Pin, Connector_PinHeader_2.54mm:PinHeader_1x02_P2.54mm_Vertical, F.Cu at (193.3, 48.8)
- added OP5: HDR 1x3 Pin, Connector_PinHeader_2.54mm:PinHeader_1x03_P2.54mm_Vertical, F.Cu at (111.0, 101.6)
- added OP6: HDR 1x3 Pin, Connector_PinHeader_2.54mm:PinHeader_1x03_P2.54mm_Vertical, F.Cu at (170.8, 95.1)
- added SPARE1: PinHeader_1x10_P2.54mm_Vertical, Connector_PinHeader_2.54mm:PinHeader_1x10_P2.54mm_Vertical, F.Cu at (108.5, 142.2)
- added SPARE2: PinHeader_2x10_P2.54mm_Vertical, Connector_PinHeader_2.54mm:PinHeader_2x10_P2.54mm_Vertical, F.Cu at (108.5, 139.7)
- added U12: 74LVC1G10, Package_TO_SOT_SMD:SOT-363_SC-70-6_Handsoldering, F.Cu at (136.5, 109.1)
- added U9: AES-MCP23S08-E/SO, Package_SO:SOIC-18W_7.5x11.6mm_P1.27mm, F.Cu at (172.5, 107.1)
- C1: value 0.1u -> T47u; footprint Capacitor_SMD:C_0603_1608Metric_Pad1.08x0.95mm_HandSolder -> Capacitor_Tantalum_SMD:CP_EIA-3528-21_Kemet-B_Pad1.50x2.35mm_HandSolder
- C10: value 47u -> 10u
- C11: value 0.1u -> 47u
- C14: value 0.1u -> 1uF
- C18: value 10u -> 1uF
- C2: value 1uF -> T47u; footprint Capacitor_SMD:C_0603_1608Metric_Pad1.08x0.95mm_HandSolder -> Capacitor_Tantalum_SMD:CP_EIA-3528-21_Kemet-B_Pad1.50x2.35mm_HandSolder
- C20: value 0.1u -> 10u
- C3: value 1uF -> 100p
- C4: value 0.1u -> 100nF
- C6: value 10u -> T47u; footprint Capacitor_SMD:C_0603_1608Metric_Pad1.08x0.95mm_HandSolder -> Capacitor_Tantalum_SMD:CP_EIA-3528-21_Kemet-B_Pad1.50x2.35mm_HandSolder
- C8: value 4.7n -> 0.1u
- C9: value 100p -> 0.1u
- D3: value LED-PWRA -> Z3.3V; footprint LED_SMD:LED_0805_2012Metric_Pad1.15x1.40mm_HandSolder -> Package_TO_SOT_SMD:SOT-23-3
- D4: value LED-PWRB -> Z24V 1W; footprint LED_SMD:LED_0805_2012Metric_Pad1.15x1.40mm_HandSolder -> Diode_SMD:D_SMA
- D5: value Z3.3V -> Z24V 1W; footprint Package_TO_SOT_SMD:SOT-23-3 -> Diode_SMD:D_SMA
- J1, J5, J6: value 1x2 Pin Hdr -> JST PH-3 2.0; footprint Connector_PinHeader_2.54mm:PinHeader_1x02_P2.54mm_Vertical -> Connector_JST:JST_PH_B3B-PH-K_1x03_P2.00mm_Vertical
- J10: value AES-Option_A-B -> Molex KK-254 AE-6410_1x03; footprint Connector_PinHeader_2.54mm:PinHeader_1x03_P2.54mm_Vertical -> Connector_Molex:Molex_KK-254_AE-6410-03A_1x03_P2.54mm_Vertical
- J11: value 1x3 Pin Hdr -> Molex KK-254 AE-6410_1x03; footprint Connector_JST:JST_PH_B3B-PH-K_1x03_P2.00mm_Vertical -> Connector_Molex:Molex_KK-254_AE-6410-03A_1x03_P2.54mm_Vertical
- J12: value 1x3 Pin Hdr -> 20-RBN; footprint Connector_Molex:Molex_SPOX_5267-03A_1x03_P2.50mm_Vertical -> Connector_PinHeader_2.54mm:PinHeader_2x10_P2.54mm_Vertical
- J13: value AES-Option_A-B -> JST-B3B-ZR 3 Pin 1.5; footprint Connector_PinHeader_2.54mm:PinHeader_1x03_P2.54mm_Vertical -> Connector_Wuerth:Wuerth_WR-WTB_64800311622_1x03_P1.50mm_Vertical
- J14: value 1x3 Pin Hdr -> Conn_01x04; footprint Connector_JST:JST_PH_B3B-PH-K_1x03_P2.00mm_Vertical -> Connector_PinHeader_2.54mm:PinHeader_1x04_P2.54mm_Vertical
- J15: value 20-RBN -> HDR 2x4 Pin Odd/Even; footprint Connector_PinHeader_2.54mm:PinHeader_2x10_P2.54mm_Vertical -> Connector_PinHeader_2.54mm:PinHeader_2x04_P2.54mm_Vertical
- J16: value 1x3 Pin Hdr -> HR-DF13_6P; footprint Connector_Molex:Molex_SPOX_5267-03A_1x03_P2.50mm_Vertical -> Connector_Hirose:Hirose_DF13-06P-1.25DSA_1x06_P1.25mm_Vertical
- J17: value 20-RBN -> HDR 1 Pin; footprint Connector_PinHeader_2.54mm:PinHeader_2x10_P2.54mm_Vertical -> Connector_PinHeader_2.54mm:PinHeader_1x01_P2.54mm_Vertical
- J18: value 1x3 Pin Hdr -> HDR 1 Pin; footprint Connector_PinHeader_2.54mm:PinHeader_1x03_P2.54mm_Vertical -> Connector_PinHeader_2.54mm:PinHeader_1x01_P2.54mm_Vertical
- J19: value 1x3 Pin Hdr -> USB-C-Conn; footprint Connector_Wuerth:Wuerth_WR-WTB_64800311622_1x03_P1.50mm_Vertical -> AES_Library:AES-USB_C-Molex-BdTopMnt-2171790001
- J2: value SERVO-BAT (10-12V) -> JST PH-3 2.0; footprint AES_Library:AES-TermBlock-2POS-5mm-Horz -> Connector_JST:JST_PH_B3B-PH-K_1x03_P2.00mm_Vertical
- J20: value 1x3 Pin Hdr -> HDR 1x2 Pin; footprint Connector_PinHeader_2.54mm:PinHeader_1x03_P2.54mm_Vertical -> Connector_PinHeader_2.54mm:PinHeader_1x02_P2.54mm_Vertical
- J21: value 1x3 Pin Hdr -> HR-DF13-6P; footprint Connector_Wuerth:Wuerth_WR-WTB_64800311622_1x03_P1.50mm_Vertical -> Connector_Hirose:Hirose_DF13-06P-1.25DSA_1x06_P1.25mm_Vertical
- J22, OP1: value 1x3 Pin Hdr -> HDR 1x3 Pin
- J23: value 1x3 Pin Hdr -> HDR 1x2 Pin; footprint Connector_Wuerth:Wuerth_WR-WTB_64800311622_1x03_P1.50mm_Vertical -> Connector_PinHeader_2.54mm:PinHeader_1x02_P2.54mm_Vertical
- J24: value Conn_01x04 -> HDR 1x2 Pin; footprint Connector_PinHeader_2.54mm:PinHeader_1x04_P2.54mm_Vertical -> Connector_PinHeader_2.54mm:PinHeader_1x02_P2.54mm_Vertical
- J25: value Conn_01x04 -> HR DF13-3P; footprint Connector_Wuerth:Wuerth_WR-WTB_64800411622_1x04_P1.50mm_Vertical -> Connector_Molex:Molex_KK-254_AE-6410-03A_1x03_P2.54mm_Vertical
- J3: value USB-C-Conn -> Molex SP-3 2.5; footprint AES_Library:AES-USB_C-Molex-BdTopMnt-2171790001 -> Connector_Molex:Molex_SPOX_5267-03A_1x03_P2.50mm_Vertical
- J4: value 1x2 Pin Hdr -> Molex SP-3 2.5; footprint Connector_PinHeader_2.54mm:PinHeader_1x02_P2.54mm_Vertical -> Connector_Molex:Molex_SPOX_5267-03A_1x03_P2.50mm_Vertical
- J7: value 1x3 Pin Hdr -> SCRW-TERM 2; footprint Connector_PinHeader_2.54mm:PinHeader_1x03_P2.54mm_Vertical -> AES_Library:AES-TermBlock-2POS-5mm-Horz
- J8: value Conn_02x04_Odd_Even -> SCRW-TERM 2; footprint Connector_PinHeader_2.54mm:PinHeader_2x04_P2.54mm_Vertical -> AES_Library:AES-TermBlock-2POS-5mm-Horz
- J9: value 1x2 Pin Hdr -> HDR 1x3 Pin; footprint Connector_PinHeader_2.54mm:PinHeader_1x02_P2.54mm_Vertical -> Connector_PinHeader_2.54mm:PinHeader_1x03_P2.54mm_Vertical
- JP1, JP2, JP3: value 1x2 Pin Hdr -> HDR 1x2 Pin
- OP2, OP3, OP4: value AES-Option_A-B -> HDR 1x3 Pin
- R1: value 0-S -> 4.7k
- R10, R11, R7, R9: value 4.7k -> 18k
- R12: value 1.78k -> 8k
- R13: value 18k -> 8k
- R14: value 560 -> 18k
- R16: value 18k -> 560
- R2, R3: value 27 -> 18k
- R4: value 4.7k -> 0-S
- R5: value 1k -> 18k
- R6: value 4.7k -> 27
- R8: value 1k -> 27
- U1: value TLV70033_SOT23-5 -> 74LS138; footprint Package_TO_SOT_SMD:SOT-23-5 -> Package_SO:TSSOP-16_4.4x5mm_P0.65mm
- U10, U8: value 74LS138 -> 74LVC2G34; footprint Package_SO:TSSOP-16_4.4x5mm_P0.65mm -> Package_TO_SOT_SMD:SOT-363_SC-70-6_Handsoldering
- U11: value 74AHCT1G125 -> 74LVC2G34; footprint Package_TO_SOT_SMD:SOT-23-5_HandSoldering -> Package_TO_SOT_SMD:SOT-363_SC-70-6_Handsoldering
- U2: value BTS51202 -> 74AHCT1G125; footprint AES_Library:AES-Inf-BTS5120-DSOP14-BP -> Package_TO_SOT_SMD:SOT-23-5_HandSoldering
- U4: value AES-MCP23S08-E/SO -> 74AHCT1G125; footprint Package_SO:SOIC-18W_7.5x11.6mm_P1.27mm -> Package_TO_SOT_SMD:SOT-23-5_HandSoldering
- U5: value 74LVC1G10 -> AES-Pico; footprint Package_TO_SOT_SMD:SOT-363_SC-70-6_Handsoldering -> AES_Library:AES-RPi_Pico_SMD_TH
- U6: value 74AHCT1G125 -> TLV70033_SOT23-5; footprint Package_TO_SOT_SMD:SOT-23-5_HandSoldering -> Package_TO_SOT_SMD:SOT-23-5
- U7: value AES-Pico -> 74LS138; footprint AES_Library:AES-RPi_Pico_SMD_TH -> Package_SO:TSSOP-16_4.4x5mm_P0.65mm
- moved J24 261.4 mm to (185.7, 46.7)
- moved D7 257.1 mm to (195.3, 55.9), turned to 180 degrees
- moved D6 255.5 mm to (195.3, 61.0), turned to 180 degrees
- moved R12 243.8 mm to (188.2, 141.2), turned to -90 degrees
- moved R13 240.1 mm to (185.2, 141.2), turned to -90 degrees
- moved C17 237.3 mm to (178.4, 50.8)
- moved C14 236.3 mm to (178.7, 56.5), turned to 90 degrees
- moved C13 236.3 mm to (175.5, 36.9), turned to -90 degrees
- moved C18 230.0 mm to (171.6, 56.5), turned to 90 degrees
- moved R15 230.0 mm to (190.3, 61.0), turned to 180 degrees
- moved R16 230.0 mm to (190.2, 55.9), turned to 180 degrees
- moved J20 223.8 mm to (178.6, 37.0)
- moved R14 205.9 mm to (161.8, 96.0), turned to 90 degrees
- moved J23 204.0 mm to (173.0, 46.7)
- moved C6 202.9 mm to (138.3, 118.4)
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Connections:
- C1 pad 1: GND -> VS-BA
- C1 pad 2: VS -> GND
- C10 pad 2: /VBUS_IF -> /VBUS_IN
- C11 pad 2: +3.3V -> /VBUS_IF
- C13 pad 1: VS -> GND
- C13 pad 2: GND -> VSYS
- C14 pad 1: /SB_TX_EN- -> VSYS
- C14 pad 2: GND -> GNDA
- C18 pad 1: GND -> +3.3VA
- C18 pad 2: /RESET- -> GNDA
- C2 pad 1: VS -> VS-BB
- C2 pad 2: GNDA -> GND
- C20 pad 1: +3.3V -> GND
- C20 pad 2: GND -> /RESET-
- C3 pad 1: +3.3VA -> GND
- C3 pad 2: GNDA -> Net-(C3-Pad2)
- C4 pad 1: +3.3VA -> VS-BA
- C4 pad 2: GNDA -> GND
- C5 pad 1: Vdrive -> VS-BB
- C6 pad 1: GND -> /RxPWR
- C6 pad 2: /VBUS_IN -> GND
- C8 pad 1: GND -> +3.3V
- C8 pad 2: VS-BB -> GND
- C9 pad 1: GND -> /SB_TX_EN-
- C9 pad 2: /SPWR_IS -> GND
- D1 pad 2: Vdrive -> VS-BA
- D2 pad 1: Net-(D1-K) -> Net-(D2-K)
- D2 pad 2: GND -> VS-BB
- D3 pad 1: GND -> /SENS_RD-
- D3 pad 2: Net-(D3-A) -> GND
- D4 pad 1: GND -> Net-(D1-K)
- D4 pad 2: Net-(D4-A) -> GND
- D5 pad 1: Net-(D5-K) -> Net-(D2-K)
- J1 pad 2: VS -> /SBA_RP
- J10 pad 1: /SBA_RP -> GND
- J10 pad 3: GND -> /SBA_RP
- J11 pad 2: /SBA_RP -> VS-BB
- J11 pad 3: /UART1_RX -> /SBB_RP
- J12 pad 2: /SBA_RP -> +3.3V
- J12 pad 3: /UART1_RX -> /S0-
- J13 pad 1: /SBB_RP -> /RxPWR
- J13 pad 2: VS-BB -> GND
- J13 pad 3: GND -> /RCVR_RX
- J14 pad 2: /SBB_RP -> /UART1_RX
- J14 pad 3: /UART1_RX -> Net-(J1-Pin_3)
- J15 pad 1: /RE_A -> GND
- J15 pad 2: +3.3V -> /RI-
- J15 pad 4: GNDA -> /DSR-
- J15 pad 5: /RE_B -> GND
- J15 pad 6: /DISP_CS- -> /DCD-
- J15 pad 8: /RESET- -> /CTS-
- J16 pad 1: GND -> +3.3V
- J16 pad 2: /SBB_RP -> Net-(J1-Pin_3)
- J17 pad 1: GND -> +3.3V
- J2 pad 2: Vdrive -> /SBA_RP
- J20 pad 2: +3.3V -> VSYS
- J21 pad 1: GND -> Net-(J21-Pin_1)
- J21 pad 2: +3.3V -> /UART0_TX
- J21 pad 3: /I2C0_SDA -> /UART0_RX
- J22 pad 2: Net-(J22-Pin_2) -> /UART0_RX
- J22 pad 3: /RCVR_RX -> /UART0_TX
- J23 pad 1: Net-(J22-Pin_2) -> GND
- J23 pad 2: GND -> +3.3V
- J24 pad 1: GND -> GNDA
- J24 pad 2: +3.3V -> +3.3VA
- J25 pad 2: +3.3V -> VSYS
- J25 pad 3: /I2C0_SCL -> /GP27A1_NEOPXL
- J4 pad 1: GNDA -> GND
- J4 pad 2: +3.3VA -> /SBA_RP
- J5 pad 2: +3.3V -> /SBB_RP
- J6 pad 2: /AUX_GP4 -> /SBB_RP
- J7 pad 2: /UART0_RX -> VS-BA
- J8 pad 2: /RI- -> VS-BB
- J9 pad 2: /AUX_GP5 -> /RxPWR
- JP1 pad 1: GND -> VS-BB
- JP1 pad 2: GNDA -> VS-BA
- JP2 pad 1: +3.3V -> Net-(J1-Pin_3)
- JP2 pad 2: +3.3VA -> /UART1_RX
- OP1 pad 1: GND -> +3.3V
- OP1 pad 2: /BD_ADDR -> /RxPWR
- OP1 pad 3: Net-(OP1-B) -> VSYS
- OP2 pad 1: /DTR- -> GND
- OP2 pad 2: /RESET- -> Net-(OP2-C)
- OP2 pad 3: GND -> /SB_TX_EN-
- OP3 pad 1: /RTS- -> /DTR-
- OP3 pad 2: /WAKEUP- -> /RESET-
- OP4 pad 1: +3.3V -> /RTS-
- OP4 pad 2: Net-(J22-Pin_2) -> /WAKEUP-
- OP4 pad 3: VS -> GND
- Q1 pad 2: VS -> VSYS
- R1 pad 1: GND -> /SENS_RD-
- R1 pad 2: Net-(J3-SHIELD-PadSH1) -> Net-(C3-Pad2)
- R10 pad 1: Net-(U2-IS) -> +3.3V
- R10 pad 2: Net-(D5-K) -> Net-(U7-E3)
- R11 pad 1: Net-(D5-K) -> +3.3V
- R11 pad 2: /SPWR_IS -> /RESET-
- R12 pad 1: Net-(U2-IS) -> /I2C0_SCL
- R12 pad 2: GND -> +3.3V
- R13 pad 1: +3.3V -> /I2C0_SDA
- R13 pad 2: Net-(OP1-B) -> +3.3V
- R14 pad 1: Net-(D6-A) -> +3.3V
- R14 pad 2: /AUX_GP4 -> Net-(OP6-B)
- R15 pad 1: Net-(D7-A) -> Net-(D6-A)
- R15 pad 2: /AUX_GP5 -> Net-(J35-Pin_2)
- R16 pad 1: +3.3V -> Net-(D7-A)
- R16 pad 2: /WAKEUP- -> Net-(J36-Pin_2)
- R2 pad 1: Net-(J3-D+-PadA6) -> +3.3V
- R2 pad 2: Net-(U3-USBDP) -> /SENS_RD-
- R3 pad 1: Net-(J3-D--PadA7) -> Net-(J1-Pin_3)
- R3 pad 2: Net-(U3-USBDM) -> +3.3V
- R4 pad 1: Net-(U4-GP0) -> GND
- R4 pad 2: Net-(U2-IN0) -> Net-(J19-SHIELD-PadSH1)
- R5 pad 1: Net-(D3-A) -> +3.3V
- R5 pad 2: VS-BA -> Net-(U1-E3)
- R6 pad 1: Net-(U4-GP1) -> Net-(J19-D+-PadA6)
- R6 pad 2: Net-(U2-IN1) -> Net-(U3-USBDP)
- R7 pad 1: Net-(U4-GP2) -> +3.3V
- R7 pad 2: Net-(U2-DEN) -> /SB_TX_EN-
- R8 pad 1: Net-(D4-A) -> Net-(J19-D--PadA7)
- R8 pad 2: VS-BB -> Net-(U3-USBDM)
- R9 pad 1: Net-(U4-GP3) -> +3.3V
- R9 pad 2: Net-(U2-DS1) -> /WAKEUP-
- U1 pad 1: VS -> /SENS_A0
- U1 pad 2: GNDA -> /SENS_A1
- U1 pad 3: VS -> /SENS_A2
- U1 pad 4: unconnected-(U1-NC-Pad4) -> GND
- U1 pad 5: +3.3VA -> GND
- U10 pad 1: /CS_A0 -> /AUX_GPO3
- U10 pad 2: /CS_A1 -> GND
- U10 pad 3: GND -> /AUX_GPO2
- U10 pad 4: GND -> Net-(J32-Pin_3)
- U10 pad 5: GND -> +3.3V
- U11 pad 1: GND -> Net-(J30-Pin_3)
- U11 pad 2: /RCVR_RX -> GND
- U11 pad 3: GND -> Net-(J31-Pin_3)
- U11 pad 4: /RCVR_IN -> /AUX_GPI1
- U2 pad 1: GND -> Net-(OP2-C)
- U2 pad 2: Net-(U2-IN0) -> /UART1_TX
- U2 pad 3: Net-(U2-DEN) -> GND
- U2 pad 4: Net-(U2-IS) -> Net-(J1-Pin_3)
- U2 pad 5: Net-(U2-DS1) -> +3.3V
- U4 pad 1: /DISP_EXP_SCK -> GND
- U4 pad 2: /DISP_EXP_MOSI -> /RCVR_RX
- U4 pad 3: /DISP_EXP_MISO -> GND
- U4 pad 4: GND -> /RCVR_IN
- U4 pad 5: GND -> +3.3V
- U5 pad 1: /EX_IRQ- -> /UART0_TX
- U5 pad 2: GND -> /UART0_RX
- U5 pad 3: /WAKEUP- -> GND
- U5 pad 4: /WU_IRQ -> /SB_TX_EN-
- U5 pad 5: +3.3V -> /WU_IRQ
- U5 pad 6: /TCH_IRQ- -> /UART1_TX
- U6 pad 1: /SB_TX_EN- -> VSYS
- U6 pad 2: /UART1_TX -> GNDA
- U6 pad 3: GND -> VSYS
- U6 pad 4: /UART1_RX -> unconnected-(U6-NC-Pad4)
- U6 pad 5: +3.3V -> +3.3VA
- U7 pad 1: /UART0_TX -> /CS_A0
- U7 pad 10: /I2C0_SCL -> unconnected-(U7-O5-Pad10)
- U7 pad 11: /CS_A0 -> unconnected-(U7-O4-Pad11)
- U7 pad 12: /RCVR_IN -> /NOCS-
- U7 pad 13: GND -> /EXIO_CS-
- U7 pad 14: /SPI1_CLK -> /TCH_CS-
- U7 pad 15: /SPI1_MOSI -> /DISP_CS-
- U7 pad 16: /SPI1_MISO -> +3.3V
- U7 pad 2: /UART0_RX -> /CS_A1
- U7 pad 4: /SB_TX_EN- -> GND
- U7 pad 5: /WU_IRQ -> GND
- U7 pad 6: /UART1_TX -> Net-(U7-E3)
- U7 pad 7: /UART1_RX -> unconnected-(U7-O7-Pad7)
- U7 pad 9: /I2C0_SDA -> unconnected-(U7-O6-Pad9)
- U8 pad 1: /SENS_A0 -> /AUX_GPO5
- U8 pad 2: /SENS_A1 -> GND
- U8 pad 3: /SENS_A2 -> /AUX_GPO4
- U8 pad 4: GND -> Net-(J35-Pin_2)
- U8 pad 5: GND -> +3.3V
- U8 pad 6: Net-(U8-E3) -> Net-(J36-Pin_2)
Routing:
- net GND: track 0.00 -> 314.6 mm, vias 0 -> 7
- net VSYS: track 0.00 -> 287.6 mm, vias 0 -> 1
- net VS-BA: track 0.00 -> 279.1 mm
- net /RESET-: track 0.00 -> 195.4 mm, vias 0 -> 2
- net GNDA: track 0.00 -> 174.3 mm
- net /SENS_RD-: track 0.00 -> 157.8 mm
- net +3.3V: track 0.00 -> 153.0 mm, vias 0 -> 7
- net /GP10_SPI1_CK: track 0.00 -> 144.7 mm
- net /GP11_SPI1_MO: track 0.00 -> 142.9 mm
- net /GP12_SPI1_MI: track 0.00 -> 140.1 mm
- net +3.3VA: track 0.00 -> 139.1 mm, vias 0 -> 1
- net /GP28A2_SWMX: track 0.00 -> 130.9 mm, vias 0 -> 3
- net /UART0_RX: track 0.00 -> 126.2 mm
- net /UART0_TX: track 0.00 -> 121.8 mm, vias 0 -> 1
- net /I2C0_SDA: track 0.00 -> 121.7 mm, vias 0 -> 2
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- added copper zone on In1.Cu, net +3.3V
- added copper zone on In2.Cu, net GND
Other:
- board outline added: 108.7 x 111.8 mm
- copper layers 2 -> 4
- board text added: "AA-P Control v1.0"
- board text added: "Copyright 2024-25 AESilky"
- board text added: "GP10"
- board text added: "GP11"
- board text added: "GP12"
- board text added: "GP14"
- board text added: "GP15"
- board text added: "GP16"
- board text added: "GP17"
- board text added: "GP18"
- board text added: "GP19"
- board text added: "GP28"
- board text added: "S P G"
