File: hw/AA_P_CtrlBd.kicad_sch (KiCad schematic)
At the start: 105 parts, among them J1 1x3 Pin Hdr, J10 1x3 Pin Hdr, J11 USB-Conn, J12 1x2 Pin Hdr, J13 1x3 Pin Hdr, J14 Conn_01x04, J15 1x2 Pin Hdr, J16 1x2 Pin Hdr, J2 1x3 Pin Hdr, J3 1x3 Pin Hdr, J4 1x3 Pin Hdr, J5 1x3 Pin Hdr, J6 1x3 Pin Hdr, J7 1x3 Pin Hdr, J8 1x3 Pin Hdr, J9 Conn_02x04_Odd_Even, J9 SERVO-BAT (6-7V), Q1 DMG2305UX, U1 AES-Pico, U2 FT231XQ, U4 ADS1015IDGS, U4 TLV70033_SOT23-5, U5 BTS51202, U6 BTS51202, U7 BTS51202, U8 BTS51202

Commit message: HW: Ready for layout.
Parts:
- removed C9 (x6): 4.7n, Capacitor_SMD:C_0603_1608Metric_Pad1.08x0.95mm_HandSolder, symbol Device:C
- removed C9 (x3): 100p, Capacitor_SMD:C_0603_1608Metric_Pad1.08x0.95mm_HandSolder, symbol Device:C
- removed C9 (x2): 0.1u, Capacitor_SMD:C_0603_1608Metric_Pad1.08x0.95mm_HandSolder, symbol Device:C
- removed D10, D14: LED-G, symbol Device:LED
- removed D11: LED-O, symbol Device:LED
- removed D12: LED-A, symbol Device:LED
- removed D13, D9: LED-Y, symbol Device:LED
- removed D3, D4, D5: 3.3V, symbol Device:D_Zener_Filled
- removed J10, J5, J6, J7, J8: 1x3 Pin Hdr, symbol Connector_Generic:Conn_01x03
- removed J14: Conn_01x04, symbol Connector_Generic:Conn_01x04
- removed J16: 1x2 Pin Hdr, symbol Connector_Generic:Conn_01x02
- removed R11: INF - ~800-80, symbol Device:R_Variable_US
- removed R6 (x13): 4.7k, Resistor_SMD:R_0805_2012Metric_Pad1.20x1.40mm_HandSolder, symbol Device:R_US
- removed R6 (x6): 1k, Resistor_SMD:R_0805_2012Metric_Pad1.20x1.40mm_HandSolder, symbol Device:R_US
- removed R6 (x3): 1.78k, Resistor_SMD:R_0805_2012Metric_Pad1.20x1.40mm_HandSolder, symbol Device:R_US
- removed R6 (x3): 18k, Resistor_SMD:R_0805_2012Metric_Pad1.20x1.40mm_HandSolder, symbol Device:R_US
- removed R6 (x2): ~, Resistor_SMD:R_0805_2012Metric_Pad1.20x1.40mm_HandSolder, symbol Device:R_US
- removed U2: FT231XQ, Package_DFN_QFN:QFN-20-1EP_4x4mm_P0.5mm_EP2.5x2.5mm, symbol Interface_USB:FT231XQ
- removed U4: ADS1015IDGS, Package_SO:TSSOP-10_3x3mm_P0.5mm, symbol Analog_ADC:ADS1015IDGS
- removed U6, U7, U8: BTS51202, symbol AES_Library:AES-BTS5120-2-2CH_PWR_SW
- added C9 (x9): 0.1u, Capacitor_SMD:C_0603_1608Metric_Pad1.08x0.95mm_HandSolder, symbol Device:C
- added D6: LED-A, LED_SMD:LED_0805_2012Metric_Pad1.15x1.40mm_HandSolder, symbol Device:LED
- added D7: LED-B, LED_SMD:LED_0805_2012Metric_Pad1.15x1.40mm_HandSolder, symbol Device:LED
- added J10, J13, OP2, OP3, OP4: AES-Option_A-B, Connector_PinHeader_2.54mm:PinHeader_1x03_P2.54mm_Vertical, symbol AES_Library:AES-Option_A-B
- added J13 (x2): 20-RBN, Connector_PinHeader_2.54mm:PinHeader_2x10_P2.54mm_Vertical, symbol Connector_Generic:Conn_02x10_Odd_Even
- added J18, J20, J22: 1x3 Pin Hdr, Connector_PinHeader_2.54mm:PinHeader_1x03_P2.54mm_Vertical, symbol Connector_Generic:Conn_01x03
- added J19, J21, J23: 1x3 Pin Hdr, Connector_Wuerth:Wuerth_WR-WTB_64800311622_1x03_P1.50mm_Vertical, symbol Connector_Generic:Conn_01x03
- added J24: Conn_01x04, Connector_PinHeader_2.54mm:PinHeader_1x04_P2.54mm_Vertical, symbol Connector_Generic:Conn_01x04
- added J25: Conn_01x04, Connector_Wuerth:Wuerth_WR-WTB_64800411622_1x04_P1.50mm_Vertical, symbol Connector_Generic:Conn_01x04
- added J5, J6, J9: 1x2 Pin Hdr, Connector_PinHeader_2.54mm:PinHeader_1x02_P2.54mm_Vertical, symbol Connector_Generic:Conn_01x02
- added R6 (x10): 18k, Resistor_SMD:R_0805_2012Metric_Pad1.20x1.40mm_HandSolder, symbol Device:R_US
- added R6 (x2): 560, Resistor_SMD:R_0805_2012Metric_Pad1.20x1.40mm_HandSolder, symbol Device:R_US
- added R6 (x3): 4.7k, Resistor_SMD:R_0805_2012Metric_Pad1.20x1.40mm_HandSolder, symbol Device:R_US
- added U10, U8: 74LS138, Package_SO:TSSOP-16_4.4x5mm_P0.65mm, symbol 74xx:74LS138
- added U11, U6: 74AHCT1G125, Package_TO_SOT_SMD:SOT-23-5_HandSoldering, symbol 74xGxx:74AHCT1G125
- added U3: FT231XS, Package_SO:SSOP-20_3.9x8.7mm_P0.635mm, symbol Interface_USB:FT231XS
- added U4: AES-MCP23S08-E/SO, Package_SO:SOIC-18W_7.5x11.6mm_P1.27mm, symbol AES_Library:AES-MCP23S08-E/SO
- added U5: 74LVC1G10, Package_TO_SOT_SMD:SOT-363_SC-70-6_Handsoldering, symbol 74xGxx:74LVC1G10
- added U9: ADS1015IDGS, Package_SO:TSSOP-10_3x3mm_P0.5mm, symbol Analog_ADC:ADS1015IDGS
- C10, C11: footprint Capacitor_SMD:C_0201_0603Metric_Pad0.64x0.40mm_HandSolder -> Capacitor_SMD:C_0603_1608Metric_Pad1.08x0.95mm_HandSolder
- D1: value SMAZ24-13-F -> Z24V 1W; footprint (none) -> Diode_SMD:D_SMA; V 24V 1W -> SMAZ24-13-F
- D2: renamed from D6; value SMAZ24-13-F -> Z24V 1W; footprint (none) -> Diode_SMD:D_SMA; V 24V 1W -> SMAZ24-13-F
- D3: renamed from D7; value LED-O -> LED-PWRA; footprint (none) -> LED_SMD:LED_0805_2012Metric_Pad1.15x1.40mm_HandSolder
- D4: renamed from D8; value LED-A -> LED-PWRB; footprint (none) -> LED_SMD:LED_0805_2012Metric_Pad1.15x1.40mm_HandSolder
- D5: renamed from D2; value 3.3V -> Z3.3V; footprint (none) -> Package_TO_SOT_SMD:SOT-23-3
- J1: renamed from J12; footprint (none) -> Connector_PinHeader_2.54mm:PinHeader_1x02_P2.54mm_Vertical
- J11: renamed from J1; footprint (none) -> Connector_JST:JST_PH_B3B-PH-K_1x03_P2.00mm_Vertical; Function Servo-LF0 -> Servo-Bus-A1
- J12: renamed from J2; footprint (none) -> Connector_Molex:Molex_SPOX_5267-03A_1x03_P2.50mm_Vertical; Function Servo-LF1 -> Servo-Bus-A2
- J14: renamed from J3; footprint (none) -> Connector_JST:JST_PH_B3B-PH-K_1x03_P2.00mm_Vertical; Function Servo-LF2 -> Servo-Bus-B1
- J16: renamed from J4; footprint (none) -> Connector_Molex:Molex_SPOX_5267-03A_1x03_P2.50mm_Vertical; Function Servo-LF3 -> Servo-Bus-B2
- J3: renamed from J11; value USB-Conn -> USB-C-Conn; footprint AES_Library:AES-USB_C_Amphenol_GSB1C4621DSHR -> AES_Library:AES-USB_C-Molex-BdTopMnt-2171790001
- J4: renamed from J15; footprint (none) -> Connector_PinHeader_2.54mm:PinHeader_1x02_P2.54mm_Vertical; Function LF_FOOT_SENS -> VA_GNDA
- J7: renamed from J13; footprint (none) -> Connector_PinHeader_2.54mm:PinHeader_1x03_P2.54mm_Vertical
- J8: renamed from J9; footprint (none) -> Connector_PinHeader_2.54mm:PinHeader_2x04_P2.54mm_Vertical
- J9: value SERVO-BAT (6-7V) -> SERVO-BAT (10-12V)
- JP1: Function RESET Connect -> SigGND-AnaGND-Conn
- JP2: Function Wake-Up Connect -> 3.3V-3.3VA-Conn
- OP1: Function PWR-SEL -> ADDR_SEL
- Q1: footprint (none) -> Package_TO_SOT_SMD:SOT-23
- U2: renamed from U5; footprint (none) -> AES_Library:AES-Inf-BTS5120-DSOP14-BP
- U7: renamed from U1; footprint RPi_Pico:RPi_Pico_SMD_TH -> AES_Library:AES-RPi_Pico_SMD_TH
Connections:
- net IS1_SEL is gone; now on net I2C0_SDA: U7.9 (GPIO6)
- net IS_EN is gone; now on net I2C0_SCL: U7.10 (GPIO7)
- net SRIS_23 is gone; now on net SPWR_IS: C9.2, R6.2
- net VSL1 is gone; now on net SBA_RP: J12.2 (Pin_2)
- net VSL3 is gone; now on net SBB_RP: J16.2 (Pin_2)
- net +3.3V: now also JP2.1 (A), C9.1, C9.2, C9.2, C9.2, C9.2, C9.2, J13.19 (Pin_19), J13.2 (Pin_2), J13.2 (Pin_2), J18.2 (Pin_2), J19.2 (Pin_2), J20.2 (Pin_2), J21.2 (Pin_2), J24.2 (Pin_2), J25.2 (Pin_2), J5.2 (Pin_2), OP4.1 (A), R6.1, R6.1, R6.1, R6.1, R6.1, R6.1, R6.1, R6.2, R6.2, R6.2, U10.16 (VCC), U11.5 (VCC), U4.18 (VDD), U5.5 (VCC), U6.5 (VCC), U8.16 (VCC), U9.8 (VDD); no longer OP1.3 (B)
- net +3.3VA: now also C9.1, J4.2 (Pin_2), JP2.2 (B), J13.11 (Pin_11); no longer OP1.1 (A)
- net CTS-: now also U3.9 (~{CTS})
- net DCD-: now also U3.8 (~{DCD})
- net DSR-: now also U3.7 (~{DSR})
- net GND: now also JP1.1 (A), OP1.1 (A), U2.1 (GND), C9.1, C9.1, C9.1, C9.1, C9.1, C9.1, C9.2, C9.2, C9.2, D6.1 (K), D7.1 (K), J10.3 (B), J13.1 (Pin_1), J13.20 (Pin_20), J13.3 (B), J13.3 (Pin_3), J13.7 (Pin_7), J18.1 (Pin_1), J19.1 (Pin_1), J20.1 (Pin_1), J21.1 (Pin_1), J22.1 (Pin_1), J23.2 (Pin_2), J24.1 (Pin_1), J25.1 (Pin_1), J5.1 (Pin_1), J6.1 (Pin_1), J9.1 (Pin_1), OP2.3 (B), OP3.3 (B), U10.3 (A2), U10.4 (E1), U10.5 (E2), U10.8 (GND), U11.1, U11.3 (GND), U3.16 (GND), U3.6 (GND), U4.4 (A1), U4.5 (A0), U4.9 (VSS), U5.2 (GND), U6.3 (GND), U8.4 (E1), U8.5 (E2), U8.8 (GND), U9.1 (ADDR), U9.3 (GND)
- net GNDA: now also JP1.2 (B), J13.4 (Pin_4)
- net I2C0_SCL: now also J18.3 (Pin_3), J19.3 (Pin_3), J24.3 (Pin_3), J25.3 (Pin_3), R6.1; no longer U7.7 (GPIO5)
- net I2C0_SDA: now also J20.3 (Pin_3), J21.3 (Pin_3), J24.4 (Pin_4), J25.4 (Pin_4), R6.1; no longer U7.6 (GPIO4)
- net RESET-: now also J13.8 (Pin_8), OP2.2 (C), R6.2, U4.6 (~{RESET}); no longer JP1.1 (A)
- net RI-: now also U3.5 (~{RI})
- net UART0_TX: now also U3.4 (RXD)
- net VS: now also C9.1, C9.2, OP4.3 (B)
- net at R6.2: now also U3.11 (USBDP)
- net VBUS_IN: now reaches C9.2, J3.A4_B9 (VBUS), J3.B4_A9 (VBUS), L1.1
- net BD_ADDR: now reaches OP1.2 (C)
- net BD_ADDR: now also U4.17 (GP7)
- net at U2.6 (IN1): now also R6.2
- net at C9.1: now also U3.13 (3V3OUT), U3.14 (~{RESET}), U3.3 (VCCIO)
- net at JP3.2 (B): now also U3.20 (TXD)
- net at R6.2: now also U3.12 (USBDM)
- net DEN: no longer names the net of U2.3 (DEN)
- net DEN: now also R6.2
- net DS1: no longer names the net of U2.5 (DS1)
- net DS1: now also R6.2
- removed net FT_SENS_LF: C9.1, J4.2 (Pin_2), U7.34 (GPIO28_ADC2)
- net FT_SENS_RT renamed SPWR_IS
- net IC_IN_1 renamed SB_TX_EN-
- net SB_TX_EN-: now also C9.1, R6.2, U6.1
- net IC_IN_2 renamed WU_IRQ
- net WU_IRQ: now also U5.4
- net IC_OUT renamed SENS_A2
- net SENS_A2: now also U8.3 (A2)
- net SRVO_PWR renamed Vdrive
- net SRV_PEN_L0 renamed DISP_EXP_SCK
- net DISP_EXP_SCK: now also J13.14 (Pin_14), U4.1 (SCK)
- net SRV_PEN_L13 renamed DISP_EXP_MISO
- net DISP_EXP_MISO: now also J13.18 (Pin_18), U4.3 (SO)
- net SRV_PEN_L2 renamed DISP_EXP_MOSI
- net DISP_EXP_MOSI: now also J13.12 (Pin_12), U4.2 (SI)
- net SRV_PEN_R0 renamed SENS_A0
- net SENS_A0: now also U8.1 (A0)
- net SRV_PEN_R1: no longer names the net of R6.1
- net SRV_PEN_R1: now also U4.10 (GP0); no longer U7.27 (GPIO21)
- net SRV_PEN_R13 renamed DISP_D/C-
- net DISP_D/C-: now also J13.10 (Pin_10)
- net SRV_PWM_L0 renamed CS_A0
- net CS_A0: now also U10.1 (A0); no longer J11.3 (Pin_3)
- net SRV_PWM_L1 renamed RCVR_IN
- net RCVR_IN: now also U11.4; no longer J12.3 (Pin_3)
- net SRV_PWM_L2 renamed SPI1_CLK
- net SPI1_CLK: now also J13.20 (Pin_20); no longer J14.3 (Pin_3)
- net SRV_PWM_L3 renamed SPI1_MOSI
- net SPI1_MOSI: now also J13.17 (Pin_17); no longer J16.3 (Pin_3)
- net SRV_PWM_R0 renamed SPI1_MISO
- net SPI1_MISO: now also J13.15 (Pin_15)
- net SRV_PWM_R1 renamed CS_A1
- net CS_A1: now also U10.2 (A1)
- net SRV_PWM_R2 renamed RE_A
- net RE_A: now also J13.1 (Pin_1)
- net SRV_PWM_R3 renamed RE_B
- net RE_B: now also J13.5 (Pin_5)
- net VBUSI renamed VBUS_IF
- net VBUS_IF: now also U3.15 (VCC)
- net VSL0 renamed SBA_RP
- net SBA_RP: now also J10.1 (A)
- net VSL2 renamed SBB_RP
- net SBB_RP: now also J13.1 (A)
- net VSR2 renamed VS-BA
- net VS-BA: now also J10.2 (C)
- net VSR3 renamed VS-BB
- net VS-BB: now also J13.2 (C)
- net WAKEUP renamed SENS_RD-
- net SENS_RD-: now also J13.10 (Pin_10), J13.12 (Pin_12), J13.14 (Pin_14), J13.16 (Pin_16), J13.18 (Pin_18), J13.4 (Pin_4), J13.6 (Pin_6), J13.8 (Pin_8), R6.2; no longer JP2.1 (A)
- new net: D6.2 (A), R6.1
- new net: OP1.3 (B), R6.2
- new net: R6.1, U4.13 (GP3)
- new net: J22.2 (Pin_2), J23.1 (Pin_1), OP4.2 (C)
- new net: R6.2, U10.6 (E3)
- new net: D7.2 (A), R6.1
- new net: R6.1, U4.11 (GP1)
- new net: R6.1, U4.12 (GP2)
- new net: R6.2, U8.6 (E3)
- new net AUX_GP4: J6.2 (Pin_2), R6.2, U4.14 (GP4)
- new net AUX_GP5: J9.2 (Pin_2), R6.2, U4.15 (GP5)
- new net DISP_BL_LED: J13.16 (Pin_16), U4.16 (GP6)
- new net DISP_CS-: J13.6 (Pin_6), U10.15 (O0)
- new net DTR-: OP2.1 (A), U3.1 (~{DTR})
- new net EXI2C_CL: U9.10 (SCL)
- new net EXI2C_DA: U9.9 (SDA)
- new net EXIO_CS-: U10.13 (O2), U4.7 (~{CS})
- new net EX_IRQ-: U4.8 (INT), U5.1
- new net NOCS-: U10.12 (O3)
- new net RCVR_RX: J22.3 (Pin_3), J23.3 (Pin_3), U11.2
- new net RTS-: OP3.1 (A), U3.2 (~{RTS})
- new net S0-: J13.3 (Pin_3), U8.15 (O0)
- new net S1-: J13.5 (Pin_5), U8.14 (O1)
- new net S2-: J13.7 (Pin_7), U8.13 (O2)
- new net S3-: J13.9 (Pin_9), U8.12 (O3)
- new net S4-: J13.11 (Pin_11), U8.11 (O4)
- new net S5-: J13.13 (Pin_13), U8.10 (O5)
- new net S6-: J13.15 (Pin_15), U8.9 (O6)
- new net S7-: J13.17 (Pin_17), U8.7 (O7)
- new net SENS_A1: U7.27 (GPIO21), U8.2 (A1)
- new net SW_MTRX: J13.9 (Pin_9), U7.34 (GPIO28_ADC2)
- new net TCH_CS-: J13.19 (Pin_19), U10.14 (O1)
- new net TCH_IRQ-: J13.13 (Pin_13), U5.6
- new net UART1_RX: J11.3 (Pin_3), J12.3 (Pin_3), J14.3 (Pin_3), J16.3 (Pin_3), R6.1, U6.4, U7.7 (GPIO5)
- new net UART1_TX: U6.2, U7.6 (GPIO4)
- new net WAKEUP-: OP3.2 (C), R6.2, U5.3
- no-connect marks 12 -> 22
Other:
- note added: "Example External I2C"
- note removed: "External (Left & Right)"
- title: Ack-Ack Legs Ctrl -> Ack-Ack Control
- moved on the sheet: C11, C9, J1, J11, J12, J14, J16, J3, J7, J8, JP3, L1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

Commit message: Sch: Remove pwr-ctrl. Add exgpio conns.
Parts:
- removed C9 (x2): 4.7n, Capacitor_SMD:C_0603_1608Metric_Pad1.08x0.95mm_HandSolder, symbol Device:C
- removed C9: 100p, Capacitor_SMD:C_0603_1608Metric_Pad1.08x0.95mm_HandSolder, symbol Device:C
- removed C9: 100nF, Capacitor_SMD:C_0603_1608Metric_Pad1.08x0.95mm_HandSolder, symbol Device:C
- removed D3: LED-PWRA, LED_SMD:LED_0805_2012Metric_Pad1.15x1.40mm_HandSolder, symbol Device:LED
- removed D4: LED-PWRB, LED_SMD:LED_0805_2012Metric_Pad1.15x1.40mm_HandSolder, symbol Device:LED
- removed J9: SERVO-BAT (10-12V), AES_Library:AES-TermBlock-2POS-5mm-Horz, symbol Connector:Screw_Terminal_01x02
- removed R6 (x6): 4.7k, Resistor_SMD:R_0805_2012Metric_Pad1.20x1.40mm_HandSolder, symbol Device:R_US
- removed R6: 1.78k, Resistor_SMD:R_0805_2012Metric_Pad1.20x1.40mm_HandSolder, symbol Device:R_US
- removed R6 (x2): 1k, Resistor_SMD:R_0805_2012Metric_Pad1.20x1.40mm_HandSolder, symbol Device:R_US
- removed U2: BTS51202, AES_Library:AES-Inf-BTS5120-DSOP14-BP, symbol AES_Library:AES-BTS5120-2-2CH_PWR_SW
- added C21, C22, C23, C24: T47u, Capacitor_Tantalum_SMD:CP_EIA-3528-21_Kemet-B_Pad1.50x2.35mm_HandSolder, symbol Device:C_Polarized_Small_US
- added C9: 100p, Capacitor_SMD:C_0603_1608Metric_Pad1.08x0.95mm_HandSolder, symbol Device:C
- added C9 (x2): 100nF, Capacitor_SMD:C_0603_1608Metric_Pad1.08x0.95mm_HandSolder, symbol Device:C
- added D3: Z3.3V, Package_TO_SOT_SMD:SOT-23-3, symbol Device:D_Zener_Filled
- added D4: Z24V 1W, Diode_SMD:D_SMA, symbol Device:D_Zener_Filled
- added J25, J30, J31, J32, J33: 1x3 Pin Hdr, Connector_Wuerth:Wuerth_WR-WTB_64800311622_1x03_P1.50mm_Vertical, symbol Connector_Generic:Conn_01x03
- added J26, J27, J28, J29: 1x3 Pin Hdr, Connector_PinHeader_2.54mm:PinHeader_1x03_P2.54mm_Vertical, symbol Connector_Generic:Conn_01x03
- added J9 (x2): SERVO-BAT (10-12V), AES_Library:AES-TermBlock-2POS-5mm-Horz, symbol Connector:Screw_Terminal_01x02
- added R6: 4.7k, Resistor_SMD:R_0805_2012Metric_Pad1.20x1.40mm_HandSolder, symbol Device:R_US
- added U10, U11, U9: 74LVC2G34, Package_TO_SOT_SMD:SOT-363_SC-70-6_Handsoldering, symbol 74xGxx:74LVC2G34
- D5: value Z3.3V -> Z24V 1W; footprint Package_TO_SOT_SMD:SOT-23-3 -> Diode_SMD:D_SMA; V (none) -> SMAZ24-13-F
- OP1: renamed from OP4; Function RRV_SEL -> Rcvr-V (Fr-Sp)
- renumbered J11 to J1, J23 to J11, J8 to J12, J3 to J13, J1 to J14, J7 to J15, J5 to J16, J4 to J17, J24 to J18, J20 to J19, J12 to J2, J21 to J20, J25 to J21, J18 to J22, J19 to J23, J14 to J3, J6 to J34, J9 to J35, J16 to J4, J22 to J7, J10 to J8, J13 to J9, JP3 to JP1, JP1 to JP3, OP1 to OP4, R1 to R3, U6 to U1, U5 to U12, U9 to U13, U8 to U2, U11 to U4, U7 to U5, U10 to U7, U4 to U8
Connections:
- net Vdrive is gone; now on net VS-BA: D1.2 (A)
- net +3.3V: now also J26.2 (Pin_2), J27.2 (Pin_2), J28.2 (Pin_2), J29.2 (Pin_2), J30.2 (Pin_2), J31.2 (Pin_2), J32.2 (Pin_2), J33.2 (Pin_2), U10.5 (VCC), U11.5 (VCC), U9.5 (VCC)
- net GND: now also C21.2, C22.2, C23.2, C24.2, C9.1, C9.2, C9.2, D3.2 (A), D4.2 (A), J25.1 (Pin_1), J26.1 (Pin_1), J27.1 (Pin_1), J28.1 (Pin_1), J29.1 (Pin_1), J30.1 (Pin_1), J31.1 (Pin_1), J32.1 (Pin_1), J33.1 (Pin_1), J9.1 (Pin_1), J9.1 (Pin_1), U10.2 (GND), U11.2 (GND), U9.2 (GND); no longer D2.2 (A)
- net SENS_RD-: now also D3.1 (K), R6.1
- net VS: now also C21.1, J25.2 (Pin_2)
- net VS-BA: now also C23.1, C9.1, J9.2 (Pin_2)
- net VS-BB: now also D2.2 (A), C24.1, C9.1, J9.2 (Pin_2)
- net AUX_GPO3: now reaches U8.13 (GP3)
- net AUX_GPO3: now also U10.3
- net at D5.1 (K): now also D2.1 (K)
- net at J11.1 (Pin_1), J7.2 (Pin_2), OP1.2 (C): now also C22.1
- net at D1.1 (K): now also D4.1 (K); no longer D2.1 (K)
- net AUX_GPI0: now reaches U8.10 (GP0)
- net AUX_GPI0: now also U11.6
- net AUX_GPI1: now reaches U8.11 (GP1)
- net AUX_GPI1: now also U11.4
- net AUX_GPO2: now reaches U8.12 (GP2)
- net AUX_GPO2: now also U10.1
- net AUX_GP4: no longer names the net of J34.2 (Pin_2), R6.2
- net AUX_GP4: now also U9.6; no longer U8.14 (GP4)
- net AUX_GP5: no longer names the net of J35.2 (Pin_2), R6.2
- net AUX_GP5: now also U9.4; no longer U8.15 (GP5)
- net SPWR_IS renamed NEOPXL
- net NEOPXL: now also J25.3 (Pin_3)
- new net: J27.3 (Pin_3), J31.3 (Pin_3), U11.3
- new net: J28.3 (Pin_3), J32.3 (Pin_3), U10.6
- new net: C9.2, R6.2
- new net: J26.3 (Pin_3), J30.3 (Pin_3), U11.1
- new net: J29.3 (Pin_3), J33.3 (Pin_3), U10.4
- new net AUX_GPO4: U8.14 (GP4), U9.1
- new net AUX_GPO5: U8.15 (GP5), U9.3
Other:
- moved on the sheet: C9, D6, D7, J34, J35, R6

Commit message: CTRL-BD-Pico: v1.0 to send for PCB.
Parts:
- removed C21: T47u, Capacitor_Tantalum_SMD:CP_EIA-3528-21_Kemet-B_Pad1.50x2.35mm_HandSolder, symbol Device:C_Polarized_Small_US
- removed J19, J22: 1x3 Pin Hdr, Connector_PinHeader_2.54mm:PinHeader_1x03_P2.54mm_Vertical, symbol Connector_Generic:Conn_01x03
- removed J20, J23, J30, J31, J32, J33: 1x3 Pin Hdr, Connector_Wuerth:Wuerth_WR-WTB_64800311622_1x03_P1.50mm_Vertical, symbol Connector_Generic:Conn_01x03
- removed J4: 1x3 Pin Hdr, Connector_Molex:Molex_SPOX_5267-03A_1x03_P2.50mm_Vertical, symbol Connector_Generic:Conn_01x03
- removed J8, J9: AES-Option_A-B, Connector_PinHeader_2.54mm:PinHeader_1x03_P2.54mm_Vertical, symbol AES_Library:AES-Option_A-B
- removed R6 (x2): 18k, Resistor_SMD:R_0805_2012Metric_Pad1.20x1.40mm_HandSolder, symbol Device:R_US
- added C22: T47u, Capacitor_Tantalum_SMD:CP_EIA-3528-21_Kemet-B_Pad1.50x2.35mm_HandSolder, symbol Device:C_Polarized_Small_US
- added H1, H2, H3, H4: M3, MountingHole:MountingHole_3.2mm_M3_ISO7380, symbol Mechanical:MountingHole
- added J10, J11, J38: Molex KK-254 AE-6410_1x03, Connector_Molex:Molex_KK-254_AE-6410-03A_1x03_P2.54mm_Vertical, symbol AES_Library:AES-Option_A-B
- added J13: HDR 2x10 Odd/Even, Connector_PinHeader_2.54mm:PinHeader_2x10_P2.54mm_Vertical, symbol Connector_Generic:Conn_02x10_Odd_Even
- added J14: Conn_01x04, Connector_PinHeader_2.54mm:PinHeader_1x04_P2.54mm_Vertical, symbol Connector_Generic:Conn_01x04
- added J16: HR-DF13_6P, Connector_Hirose:Hirose_DF13-06P-1.25DSA_1x06_P1.25mm_Vertical, symbol Connector_Generic:Conn_01x06
- added J17, J18: HDR 1 Pin, Connector_PinHeader_2.54mm:PinHeader_1x01_P2.54mm_Vertical, symbol Connector_Generic:Conn_01x01
- added J2, J6: JST PH-3 2.0, Connector_JST:JST_PH_B3B-PH-K_1x03_P2.00mm_Vertical, symbol Connector_Generic:Conn_01x03
- added J21: HR-DF13-6P, Connector_Hirose:Hirose_DF13-06P-1.25DSA_1x06_P1.25mm_Vertical, symbol Connector_Generic:Conn_01x06
- added J28: HR-DF13-4P 1.25, Connector_Hirose:Hirose_DF13-04P-1.25DSA_1x04_P1.25mm_Vertical, symbol Connector_Generic:Conn_01x04
- added J3: Molex SP-3 2.5, Connector_Molex:Molex_SPOX_5267-03A_1x03_P2.50mm_Vertical, symbol Connector_Generic:Conn_01x03
- added J37: HDR 1x10, Connector_PinHeader_2.54mm:PinHeader_1x10_P2.54mm_Vertical, symbol Connector_Generic:Conn_01x10
- added JP1, JP2: HDR 1x2 Pin, Connector_PinHeader_2.54mm:PinHeader_1x02_P2.54mm_Vertical, symbol Jumper:Jumper_2_Open
- added OP2, OP5: HDR 1x3 Pin, Connector_PinHeader_2.54mm:PinHeader_1x03_P2.54mm_Vertical, symbol AES_Library:AES-Option_A-B
- added R6 (x2): 8k, Resistor_SMD:R_0805_2012Metric_Pad1.20x1.40mm_HandSolder, symbol Device:R_US
- D6: renamed from D7; value LED-B -> LED-A
- D7: renamed from D6; value LED-A -> LED-B
- J1: value 1x3 Pin Hdr -> JST PH-3 2.0; Function Servo-Bus-A1 -> Servo-BusA1
- J13: value 20-RBN -> HDR 2x10 Odd/Even
- J13: renamed from J11; value 1x3 Pin Hdr -> JST-B3B-ZR 3 Pin 1.5
- J15: renamed from J12; value Conn_02x04_Odd_Even -> HDR 2x4 Pin Odd/Even
- J20: renamed from J14; value 1x2 Pin Hdr -> HDR 1x2 Pin
- J22: renamed from J15; value 1x3 Pin Hdr -> HDR 1x3 Pin
- J23: renamed from J16; value 1x2 Pin Hdr -> HDR 1x2 Pin
- J24: renamed from J17; value 1x2 Pin Hdr -> HDR 1x2 Pin
- J25: value 1x3 Pin Hdr -> HR DF13-3P; footprint Connector_Wuerth:Wuerth_WR-WTB_64800311622_1x03_P1.50mm_Vertical -> Connector_Molex:Molex_KK-254_AE-6410-03A_1x03_P2.54mm_Vertical
- J26: renamed from J18; value Conn_01x04 -> HDR 1x4 Pin
- J27: renamed from J21; value Conn_01x04 -> JST-B4B-ZR 4P 1.5
- J30: renamed from J26; value 1x3 Pin Hdr -> HDR 1x3 Pin; Function AGPI_0A -> AGPI_0
- J31: renamed from J27; value 1x3 Pin Hdr -> HDR 1x3 Pin; Function AGPI_1A -> AGPI_1
- J32: renamed from J29; value 1x3 Pin Hdr -> HDR 1x3 Pin; Function AGPO_3A -> AGPO_2
- J33: renamed from J28; value 1x3 Pin Hdr -> HDR 1x3 Pin; Function AGPO_2A -> AGPO_3
- J35: value 1x2 Pin Hdr -> HR DF13-2P; footprint Connector_PinHeader_2.54mm:PinHeader_1x02_P2.54mm_Vertical -> Connector_Hirose:Hirose_DF13-02P-1.25DSA_1x02_P1.25mm_Vertical; Function AUX_GP5 -> AGPO_4
- J36: renamed from J34; value 1x2 Pin Hdr -> HR DF13-2P; footprint Connector_PinHeader_2.54mm:PinHeader_1x02_P2.54mm_Vertical -> Connector_Hirose:Hirose_DF13-02P-1.25DSA_1x02_P1.25mm_Vertical; Function AUX_GP4 -> AGP0_5
- J4: renamed from J2; value 1x3 Pin Hdr -> Molex SP-3 2.5; Function Servo-Bus-A2 -> Servo-BusA4
- J5: renamed from J3; value 1x3 Pin Hdr -> JST PH-3 2.0; Function Servo-Bus-B1 -> Servo-BusB1
- J9: value SERVO-BAT (10-12V) -> SCRW-TERM 2; Function (none) -> SERVO-BAT (6-8V or 10-12V)
- J9: renamed from J7; value 1x3 Pin Hdr -> HDR 1x3 Pin
- JP3: renamed from JP1; value 1x2 Pin Hdr -> HDR 1x2 Pin
- JP4: renamed from JP2; value 1x2 Pin Hdr -> HDR 1x2 Pin
- JP5: renamed from JP3; value 1x2 Pin Hdr -> HDR 1x2 Pin
- OP1: value AES-Option_A-B -> HDR 1x3 Pin
- OP3: renamed from OP2; value AES-Option_A-B -> HDR 1x3 Pin; Function (none) -> Reset Ctrl
- OP4: renamed from OP3; value AES-Option_A-B -> HDR 1x3 Pin; Function (none) -> Wakeup Ctrl
- OP6: renamed from OP4; value 1x3 Pin Hdr -> HDR 1x3 Pin
- Q1: symbol AES_Library:AES-DMG2305UX -> AES_Library:DMG2305UX-AES; Function (none) -> VBUS Input Gate
- renumbered C23 to C1, C24 to C2, C22 to C6, J13 to J19, R3 to R4, U2 to U1, U1 to U2, U9 to U8, U8 to U9
Connections:
- net +3.3V: now also J14.4 (Pin_4), J16.1 (Pin_1), J17.1 (Pin_1), OP5.1 (A), R6.2, R6.2
- net AUX_GPO2: now also U10.3; no longer U10.1
- net AUX_GPO3: now also U10.1; no longer U10.3
- net AUX_GPO4: now also U8.3; no longer U8.1
- net AUX_GPO5: now also U8.1; no longer U8.3
- net DCD-: now also J15.6 (Pin_6); no longer J15.4 (Pin_4)
- net DSR-: now also J15.4 (Pin_4); no longer J15.6 (Pin_6)
- net GND: now also C22.2, J10.1 (A), J11.1 (A), J14.1 (Pin_1), J16.6 (Pin_6), J18.1 (Pin_1), J2.1 (Pin_1), J21.6 (Pin_6), J28.4 (Pin_4), J3.1 (Pin_1), J37.1 (Pin_1), J37.10 (Pin_10), J37.2 (Pin_2), J37.3 (Pin_3), J37.4 (Pin_4), J37.5 (Pin_5), J37.6 (Pin_6), J37.7 (Pin_7), J37.8 (Pin_8), J37.9 (Pin_9), J38.1 (A), J6.1 (Pin_1), OP2.1 (A)
- net I2C0_SCL: now also J28.2 (Pin_2), R6.1
- net I2C0_SDA: now also J28.3 (Pin_3), R6.1
- net SBA_RP: now also J10.3 (B), J2.2 (Pin_2), J3.2 (Pin_2)
- net SBB_RP: now also J11.3 (B), J6.2 (Pin_2)
- net SB_TX_EN-: now also OP2.3 (B); no longer U2.1
- net UART0_RX: now also J21.3 (Pin_3)
- net UART0_TX: now also J21.2 (Pin_2)
- net UART1_RX: now also J14.2 (Pin_2), J16.3 (Pin_3), JP2.2 (B); no longer J1.3 (Pin_3), J4.3 (Pin_3), J5.3 (Pin_3), R6.1, U2.4
- net VS-BA: now also J10.2 (C), J38.2 (C), JP1.2 (B)
- net VS-BB: now also J11.2 (C), JP1.1 (A)
- net RxPWR: now reaches C6.1, J13.1 (Pin_1), J9.2 (Pin_2), OP1.2 (C)
- net DISP_BL_LED renamed AGP6_DISPBL
- net DISP_D/C- renamed GP17_D_D/C-
- net GP17_D_D/C-: now also J13.14 (Pin_14)
- net DISP_EXP_MISO renamed GP16_DE_MISO
- net GP16_DE_MISO: now also J13.12 (Pin_12)
- net DISP_EXP_MOSI renamed GP19_DE_MOSI
- net GP19_DE_MOSI: now also J13.18 (Pin_18)
- net DISP_EXP_SCK renamed GP18_DE_SCK
- net GP18_DE_SCK: now also J13.16 (Pin_16)
- net NEOPXL renamed GP27A1_NEOPXL
- net RE_A renamed GP14_RE_A
- net GP14_RE_A: now also J13.8 (Pin_8)
- net RE_B renamed GP15_RE_B
- net GP15_RE_B: now also J13.10 (Pin_10)
- net SPI1_CLK renamed GP10_SPI1_CK
- net GP10_SPI1_CK: now also J13.2 (Pin_2)
- net SPI1_MISO renamed GP12_SPI1_MI
- net GP12_SPI1_MI: now also J13.6 (Pin_6)
- net SPI1_MOSI renamed GP11_SPI1_MO
- net GP11_SPI1_MO: now also J13.4 (Pin_4)
- net SW_MTRX renamed GP28A2_SWMX
- net GP28A2_SWMX: now also J13.20 (Pin_20)
- net VS renamed VSYS
- net VSYS: now also C22.1, J28.1 (Pin_1), OP5.3 (B)
- new net: OP2.2 (C), U2.1
- new net: J1.3 (Pin_3), J14.3 (Pin_3), J16.2 (Pin_2), J2.3 (Pin_3), J3.3 (Pin_3), J4.3 (Pin_3), J5.3 (Pin_3), J6.3 (Pin_3), JP2.1 (A), R6.1, U2.4
- new net: J21.1 (Pin_1), OP5.2 (C)
- new net SBC_RP: J13.1 (Pin_1), J13.11 (Pin_11), J13.13 (Pin_13), J13.15 (Pin_15), J13.17 (Pin_17), J13.19 (Pin_19), J13.3 (Pin_3), J13.5 (Pin_5), J13.7 (Pin_7), J13.9 (Pin_9), J38.3 (B)
- no-connect marks 22 -> 26
Other:
- moved on the sheet: C6, C9, D6, D7, J1, J13, J22, J26, J27, J32, J33, J35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

Commit message: HW: Add pdf schematic of the Pico Ctrl board.
Parts:
- added R17: 18k, symbol Device:R
Connections:
- net +3.3V: now also R17.1
- net TCH_IRQ-: now also R17.2
Other:
- note added: "Add Pull-Up for when display isn't connected"
- note added: "DO NOT POPULATE C9"
Changed lines of the file:
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@@
     (title "Ack-Ack Control")
     (date "2024-11-03")
-    (rev "1.0")
+    (rev "1.0a")
     (company "SilkyDESIGN - AESilky")
     (comment 1 "Copyright 2024 AESilky")
+    (comment 3 "a: Change Order for v1.0 boards")
   )
   (junction (at 250.19 300.99) (diameter 0) (color 0 0 0 0)
@@
   (junction (at 140.97 190.5) (diameter 0) (color 0 0 0 0)
   )
+  (junction (at 307.34 154.94) (diameter 0) (color 0 0 0 0)
+  )
   (junction (at 182.88 165.1) (diameter 0) (color 0 0 0 0)
   )
@@
   (junction (at 245.11 223.52) (diameter 0) (color 0 0 0 0)
   )
+  (junction (at 318.77 143.51) (diameter 0) (color 0 0 0 0)
+  )
   (junction (at 394.97 175.26) (diameter 0) (color 0 0 0 0)
   )
@@
     (stroke (width 0) (type default))
   )
-  (wire (pts (xy 285.75 154.94) (xy 359.41 154.94))
+  (wire (pts (xy 285.75 154.94) (xy 307.34 154.94))
     (stroke (width 0) (type default))
   )
@@
     (stroke (width 0) (type default))
   )
+  (wire (pts (xy 307.34 143.51) (xy 318.77 143.51))
+    (stroke (width 0) (type default))
+  )
   (wire (pts (xy 45.72 107.95) (xy 45.72 109.22))
     (stroke (width 0) (type default))
@@
     (stroke (width 0) (type default))
   )
+  (wire (pts (xy 307.34 152.4) (xy 307.34 154.94))
+    (stroke (width 0) (type default))
+  )
   (wire (pts (xy 179.07 205.74) (xy 309.88 205.74))
     (stroke (width 0) (type default))
@@
     (stroke (width 0) (type default))
   )
+  (wire (pts (xy 318.77 143.51) (xy 318.77 190.5))
+    (stroke (width 0) (type default))
+  )
   (wire (pts (xy 30.48 177.8) (xy 30.48 187.96))
     (stroke (width 0) (type default))
@@
     (stroke (width 0) (type default))
   )
+  (wire (pts (xy 99.06 181.61) (xy 101.6 179.07))
+    (stroke (width 0) (type default) (color 255 0 0 1))
+  )
   (wire (pts (xy 182.88 153.67) (xy 186.69 153.67))
     (stroke (width 0) (type default))
@@
     (stroke (width 0) (type default))
   )
+  (wire (pts (xy 307.34 143.51) (xy 307.34 144.78))
+    (stroke (width 0) (type default))
+  )
   (wire (pts (xy 55.88 265.43) (xy 55.88 267.97))
     (stroke (width 0) (type default))
@@
     (stroke (width 0) (type default))
   )
+  (wire (pts (xy 99.06 179.07) (xy 101.6 181.61))
+    (stroke (width 0) (type default) (color 255 0 0 1))
+  )
   (wire (pts (xy 355.6 187.96) (xy 355.6 200.66))
     (stroke (width 0) (type default))
@@
     (stroke (width 0) (type default))
   )
-  (wire (pts (xy 318.77 151.13) (xy 318.77 190.5))
+  (wire (pts (xy 318.77 139.7) (xy 318.77 143.51))
     (stroke (width 0) (type default))
   )
@@
     (stroke (width 0) (type default))
   )
+  (wire (pts (xy 307.34 154.94) (xy 359.41 154.94))
+    (stroke (width 0) (type default))
+  )
   (wire (pts (xy 389.89 130.81) (xy 389.89 128.27))
     (stroke (width 0) (type default))
@@
     (effects (font (size 1.27 1.27)) (justify left top))
   )
+  (text "DO NOT\nPOPULATE\nC9" (at 91.44 185.42 0)
+    (effects (font (size 1.27 1.27) (color 255 0 0 1)) (justify left bottom))
+  )
   (text "Example External I2C" (at 377.19 278.13 0)
     (effects (font (size 1.27 1.27)) (justify left bottom))
@@
   (text "NOTE: Must remove\nPico R7 200R, so\n3.3V is disconnected\nfrom ADC_VREF"
     (at 162.56 53.34 0)
-    (effects (font (size 1.27 1.27) (thickness 0.254) bold (color 255 0 0 1)) (justify left bottom))
+    (effects (font (size 1.27 1.27) (thickness 0.254) bold (color 194 0 0 1)) (justify left bottom))
   )
   (text "(~5V)" (at 57.15 264.16 0)
     (effects (font (size 1.27 1.27) (color 0 0 194 1)) (justify left bottom))
   )
+  (text "Add Pull-Up\nfor when display\nisn't connected" (at 298.45 142.24 0)
+    (effects (font (size 1.27 1.27) (color 255 0 0 1)) (justify left bottom))
+  )
   (label "GP14_RE_A" (at 364.49 182.88 0) (fields_autoplaced)
     (effects (font (size 1.27 1.27)) (justify left bottom))
@@
     )
   )
-  (symbol (lib_id "power:+3.3V") (at 318.77 151.13 0) (mirror y) (unit 1)
+  (symbol (lib_id "power:+3.3V") (at 318.77 139.7 0) (mirror y) (unit 1)
     (in_bom yes) (on_board yes) (dnp no)
-    (property "Reference" "#PWR028" (at 318.77 154.94 0)
+    (property "Reference" "#PWR028" (at 318.77 143.51 0)
       (effects (font (size 1.27 1.27)) hide)
     )
-    (property "Value" "+3.3V" (at 318.77 147.32 0)
+    (property "Value" "+3.3V" (at 318.77 135.89 0)
       (effects (font (size 1.27 1.27)))
     )
-    (property "Footprint" "" (at 318.77 151.13 0)
+    (property "Footprint" "" (at 318.77 139.7 0)
       (effects (font (size 1.27 1.27)) hide)
     )
-    (property "Datasheet" "" (at 318.77 151.13 0)
+    (property "Datasheet" "" (at 318.77 139.7 0)
       (effects (font (size 1.27 1.27)) hide)
     )
@@
         )
       )
+    )
+  )
+  (symbol (lib_id "Device:R") (at 307.34 148.59 0) (unit 1)
+    (in_bom yes) (on_board yes) (dnp no) (fields_autoplaced)
+    (property "Reference" "R17" (at 309.88 147.955 0)
+      (effects (font (size 1.27 1.27)) (justify left))
+    )
+    (property "Value" "18k" (at 309.88 150.495 0)
+      (effects (font (size 1.27 1.27)) (justify left))
+    )
+    (property "Footprint" "" (at 305.562 148.59 90)
+      (effects (font (size 1.27 1.27)) hide)
+    )
+    (property "Datasheet" "~" (at 307.34 148.59 0)
+      (effects (font (size 1.27 1.27)) hide)
+    )
+    (pin "1")
+    (pin "2")
+    (instances
+      (project "AA_P_CtrlBd"
+        (path "/349a4f05-da1f-46bd-b554-d51220f02229"
+          (reference "R17") (unit 1)
+        )
+      )
