File: hw/AA_PwrSens_Dist.kicad_sch (KiCad schematic)
At the start: 100 parts, among them J1 Conn_01x03, J10 Barrel_Jack_Switch, J11 Conn_01x03, J12 Screw_Terminal_01x02, J13 20-RBN, J13 Screw_Terminal_01x02, J14 Screw_Terminal_01x02, J15 Conn_01x04, J17 HDR 1x3 Pin, J18 Conn_01x02, J19 Conn_01x02, J2 Conn_01x03, J20 Conn_01x02, J21 HDR 1x3 Pin, J22 HDR 1x3 Pin, J23 HDR 1x3 Pin, J24 Conn_01x04, J25 HDR 1x3 Pin, J26 Conn_01x02, J27 Conn_01x04, J28 HDR 1x3 Pin, J29 Conn_01x02, J3 Conn_01x03, J30 Conn_01x05, J31 HDR 1x3 Pin, J4 Conn_01x03, J5 Conn_01x03, J6 Conn_01x04, J7 Screw_Terminal_01x02, J8 Screw_Terminal_01x02, J9 Screw_Terminal_01x02, U1 ADS1015IDGS, U2 74AHCT1G125, U3 74AHCT1G125, U4 74AHCT1G125, U5 74AHCT1G125, U6 74AHCT1G125, U7 BTS51202, U8 24LC32, U9 TLV70033_SOT23-5

Commit message: PCB: Files for PCB rev 1.0
Parts:
- removed J21, J22: HDR 1x3 Pin, Connector_PinHeader_2.54mm:PinHeader_1x03_P2.54mm_Vertical, symbol Connector_Generic:Conn_01x03
- added C9: 0.1u, Capacitor_SMD:C_0603_1608Metric_Pad1.08x0.95mm_HandSolder, symbol Device:C
- added D11: BZV55C3V3, Diode_SMD:D_MiniMELF, symbol Diode:BZV55C3V3
- added H1, H10, H11, H2, H3, H4, H5, H6, H7, H8, H9: MountingHole, MountingHole:MountingHole_3.2mm_M3, symbol Mechanical:MountingHole
- added J11, J13: JST-PH-B4B, Connector_JST:JST_PH_B4B-PH-K_1x04_P2.00mm_Vertical, symbol Connector_Generic:Conn_01x04
- added J28: JST-PH-B3B, Connector_JST:JST_PH_B3B-PH-K_1x03_P2.00mm_Vertical, symbol Connector_Generic:Conn_01x03
- added J29, J30, J34, J35, J36, J37: Molex KK-254 AE-6410_1x03, Connector_Molex:Molex_KK-254_AE-6410-03A_1x03_P2.54mm_Vertical, symbol Connector_Generic:Conn_01x03
- added J41: JST-PH-B2B, Connector_JST:JST_PH_B2B-PH-K_1x02_P2.00mm_Vertical, symbol Connector_Generic:Conn_01x02
- added J42, J43, J44: Conn_01x02, Connector_JST:JST_PH_B2B-PH-K_1x02_P2.00mm_Vertical, symbol Connector_Generic:Conn_01x02
- added PS5: DC-DC-Mod-1117, AES_Library:DC-DC_Module-SM-44_100-AES, symbol AES_Library:DC-DC-Mod-1117-AES
- added TP1: 1-Pin, Connector_PinHeader_2.54mm:PinHeader_1x01_P2.54mm_Vertical, symbol Test_point_Jump:TP_01
- C2, C3: footprint (none) -> Capacitor_THT:CP_Radial_D16.0mm_P7.50mm; PN EV1H332MNN18P1F8 -> EKYC500ELL162ML25S
- C9: now in the parts list
- J1: renamed from J6; value Conn_01x04 -> JST-PH-B4B
- J10: footprint (none) -> Connector_BarrelJack:BarrelJack_Kycon_KLDX-0202-xC_Horizontal
- J12: renamed from J11; value Conn_01x03 -> JST-VH-B3P; footprint (none) -> Connector_JST:JST_VH_B3P-VH-B_1x03_P3.96mm_Vertical
- J14: renamed from J30; footprint (none) -> Connector_PinHeader_2.54mm:PinHeader_1x05_P2.54mm_Vertical
- J15: renamed from J27; value Conn_01x04 -> JST-PH-B4B; footprint (none) -> Connector_JST:JST_PH_B4B-PH-K_1x04_P2.00mm_Vertical
- J16: renamed from J28; value HDR 1x3 Pin -> JST-PH-B3B; footprint Connector_PinHeader_2.54mm:PinHeader_1x03_P2.54mm_Vertical -> Connector_JST:JST_PH_B3B-PH-K_1x03_P2.00mm_Vertical
- J17: renamed from J15; value Conn_01x04 -> JST-VH-455-B4P; footprint (none) -> Connector_JST:JST_VH_B4P-VH_1x04_P3.96mm_Vertical
- J18: renamed from J29; value Conn_01x02 -> JST-PH-B2B; footprint (none) -> Connector_JST:JST_PH_B2B-PH-K_1x02_P2.00mm_Vertical
- J19: renamed from J12; value Screw_Terminal_01x02 -> SCRW-TERM-2; footprint (none) -> AES_Library:AES-TermBlock-2POS-5mm-Horz
- J2: renamed from J1; footprint (none) -> Connector_PinHeader_2.54mm:PinHeader_1x03_P2.54mm_Vertical
- J20: renamed from J13; value Screw_Terminal_01x02 -> SCRW-TERM-2; footprint (none) -> AES_Library:AES-TermBlock-2POS-5mm-Horz
- J21: renamed from J14; value Screw_Terminal_01x02 -> SCRW-TERM-2; footprint (none) -> AES_Library:AES-TermBlock-2POS-5mm-Horz
- J23: renamed from J17; value HDR 1x3 Pin -> AGPIO-PWRCTRL
- J24: renamed from J18; footprint (none) -> Connector_PinHeader_2.54mm:PinHeader_1x02_P2.54mm_Vertical
- J25: renamed from J19; footprint (none) -> Connector_PinHeader_2.54mm:PinHeader_1x02_P2.54mm_Vertical
- J27: renamed from J24; value Conn_01x04 -> JST-PH-B4B
- J3: renamed from J2; footprint (none) -> Connector_PinHeader_2.54mm:PinHeader_1x03_P2.54mm_Vertical
- J31: renamed from J23; value HDR 1x3 Pin -> Molex KK-254 AE-6410_1x03; footprint Connector_PinHeader_2.54mm:PinHeader_1x03_P2.54mm_Vertical -> Connector_Molex:Molex_KK-254_AE-6410-03A_1x03_P2.54mm_Vertical
- J32: renamed from J26; value Conn_01x02 -> JST-PH-B2B; footprint (none) -> Connector_JST:JST_PH_B2B-PH-K_1x02_P2.00mm_Vertical
- J33: renamed from J25; value HDR 1x3 Pin -> JST-PH-B3B
- J38: renamed from J31; value HDR 1x3 Pin -> JST-PH-B3B
- J4: renamed from J3; footprint (none) -> Connector_PinHeader_2.54mm:PinHeader_1x03_P2.54mm_Vertical
- J5: renamed from J4; footprint (none) -> Connector_PinHeader_2.54mm:PinHeader_1x03_P2.54mm_Vertical
- J6: renamed from J5; footprint (none) -> Connector_PinHeader_2.54mm:PinHeader_1x03_P2.54mm_Vertical
- J7, J8, J9: value Screw_Terminal_01x02 -> ScrewLug-2; footprint (none) -> TerminalBlock_Dinkle:TerminalBlock_Dinkle_DT-55-B01X-02_P10.00mm; PN (none) -> OST-OSTYK51102030
- Opt-A1, Opt-P1: footprint (none) -> Connector_PinHeader_2.54mm:PinHeader_1x03_P2.54mm_Vertical
- Opt-A2: footprint (none) -> Connector_PinHeader_2.54mm:PinHeader_1x02_P2.54mm_Vertical
- R1: renamed from R2; value 20k -> 10k
- U1: footprint Package_SO:TSSOP-10_3x3mm_P0.5mm -> Package_SO:VSSOP-10_3x3mm_P0.5mm; now in the parts list
- renumbered D17 to D12, D11 to D13, D12 to D14, D13 to D15, D14 to D16, D15 to D17, D16 to D18, D18 to D19, J20 to J26, R23 to R14, R24 to R15, R1 to R2
Connections:
- net +3.3V: now also C9.1, PS5.3 (OUT+)
- net +5V: now also J29.3 (Pin_3), J30.3 (Pin_3), J42.2 (Pin_2), J43.2 (Pin_2), PS5.1 (IN+)
- net +5VD: now also J27.3 (Pin_3), J32.2 (Pin_2), J38.2 (Pin_2), J28.2 (Pin_2), J34.3 (Pin_3), J35.3 (Pin_3), J41.2 (Pin_2), J44.2 (Pin_2); no longer J27.4 (Pin_4), J32.1 (Pin_1), J33.1 (Pin_1), J38.1 (Pin_1)
- net AIN0: now also D11.1 (K), J11.1 (Pin_1); no longer D9.1 (K), R7.2, R9.1
- net AIN1: now also J11.2 (Pin_2); no longer R10.1, R8.2
- net AIN2: now also D9.1 (K), J11.3 (Pin_3); no longer C9.2, R6.2
- net GND: now also J27.4 (Pin_4), J32.1 (Pin_1), C9.2, D11.2 (A), J11.4 (Pin_4), J13.4 (Pin_4), J28.1 (Pin_1), J29.1 (Pin_1), J30.1 (Pin_1), J34.1 (Pin_1), J35.1 (Pin_1), J36.1 (Pin_1), J37.1 (Pin_1), J41.1 (Pin_1), J42.1 (Pin_1), J43.1 (Pin_1), J44.1 (Pin_1), PS5.2 (IN-), PS5.4 (OUT-); no longer J27.3 (Pin_3), J32.2 (Pin_2), J38.2 (Pin_2)
- net V12_C1: now also J36.2 (Pin_2), J36.3 (Pin_3)
- net V7_C: now also J37.2 (Pin_2), J37.3 (Pin_3)
- net at R1.2, U1.2 (ALERT/RDY): now also TP1.1 (Pin_1)
- new net: J33.1 (Pin_1), J38.1 (Pin_1)
- new net: J13.1 (Pin_1), R7.2, R9.1
- new net: J13.2 (Pin_2), R10.1, R8.2
- new net: C9.2, J13.3 (Pin_3), R6.2
- no-connect marks 13 -> 18
Other:
- added sheet AA-HeadCtrl (aa-headctrl.kicad_sch)
- note added: "Board to Board Power Connections"
- note added: "Optional Module rather than regulator"
- moved on the sheet: C9, D12, D19, J1, J14, J2, J21, J27, J32, J33, J38, Opt-A1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
